File: weeSpindel.sch (KiCad schematic (older format))
At the start: 21 parts, among them J1 POWER, J2 MPU-6050, U1 ESP-12E, U2 HT7733SA, U3 DS18B20

Commit message: add a calibrate jumper
Parts:
- added JP1: Cal, CPB:Socket_Strip_Straight_1x02_Oval_Pitch2.54mm, symbol Device:Jumper
Connections:
- net labels added: DQ
- net labels removed: GPIO12
- wire segments 87 -> 90
- no-connect marks 8 -> 7
Changed lines of the file:
@@
 EESchema Schematic File Version 4
-LIBS:ESP_Single_A-cache
+LIBS:weeSpindel-cache
 EELAYER 26 0
 EELAYER END
@@
 	2300 6950 2300 7000
 Wire Wire Line
-	900  7000 2300 7000
+	900  7000 1300 7000
 Connection ~ 2300 7000
 Wire Wire Line
@@
 $EndComp
 Text GLabel 1300 6250 0    50   Input ~ 0
-GPIO12
+DQ
 Wire Wire Line
 	6950 2500 7150 2500
@@
 $EndComp
 Text GLabel 6450 5150 2    50   Input ~ 0
-GPIO12
+DQ
 $Comp
 L power:GND #PWR05
@@
 Wire Wire Line
 	1300 6250 1400 6250
-NoConn ~ 1400 6350
+Wire Wire Line
+	1300 6350 1400 6350
+$Comp
+L Device:Jumper JP1
+U 1 1 5E859075
+P 1300 6650
+F 0 "JP1" V 1346 6562 50  0000 R CNN
+F 1 "Cal" V 1255 6562 50  0000 R CNN
+F 2 "CPB:Socket_Strip_Straight_1x02_Oval_Pitch2.54mm" H 1300 6650 50  0001 C CNN
+F 3 "~" H 1300 6650 50  0001 C CNN
+	1    1300 6650
+	0    -1   -1   0
+$EndComp
+Wire Wire Line
+	1300 6950 1300 7000
+Connection ~ 1300 7000
+Wire Wire Line
+	1300 7000 2300 7000
 $EndSCHEMATC

Commit message: now with integrated battery, power switch.
Parts:
- removed J1: POWER, CPB:Socket_Strip_Straight_1x02_Oval_Pitch2.54mm, symbol Connector_Generic:Conn_01x02
- added BT1: AA, CPB:Battery_Springs_AA, symbol Device:Battery_Cell
- added SW1: POWER, CPB:SPST Switch 9mmx3.5mm C223839, symbol Switch:SW_SPST
Connections:
- wire segments 90 -> 93
Other:
- moved on the sheet: JP1
Changed lines of the file:
@@
 Wire Wire Line
 	2300 6950 2300 7000
-Wire Wire Line
-	900  7000 1300 7000
 Connection ~ 2300 7000
 Wire Wire Line
@@
 	1650 2100 1700 2100
 Connection ~ 1650 2100
-Text GLabel 2200 800  0    50   Input ~ 0
+Text GLabel 1950 1050 2    50   Output ~ 0
 VBAT
 Text GLabel 1050 2100 0    50   Input ~ 0
@@
 Wire Wire Line
 	1650 3050 2600 3050
-$Comp
-L Connector_Generic:Conn_01x02 J1
-U 1 1 5D26FFDF
-P 2600 900
-F 0 "J1" H 2680 892 50  0000 L CNN
-F 1 "POWER" H 2680 801 50  0000 L CNN
-F 2 "CPB:Socket_Strip_Straight_1x02_Oval_Pitch2.54mm" H 2600 900 50  0001 C CNN
-F 3 "~" H 2600 900 50  0001 C CNN
-	1    2600 900
-	1    0    0    1
-$EndComp
 Wire Wire Line
 	3700 2400 3700 2100
@@
 L power:GND #PWR01
 U 1 1 5DBBA683
-P 2050 900
-F 0 "#PWR01" H 2050 650 50  0001 C CNN
-F 1 "GND" H 2055 727 50  0000 C CNN
-F 2 "" H 2050 900 50  0001 C CNN
-F 3 "" H 2050 900 50  0001 C CNN
-	1    2050 900
+P 900 1300
+F 0 "#PWR01" H 900 1050 50  0001 C CNN
+F 1 "GND" H 905 1127 50  0000 C CNN
+F 2 "" H 900 1300 50  0001 C CNN
+F 3 "" H 900 1300 50  0001 C CNN
+	1    900  1300
 	1    0    0    -1
 $EndComp
@@
 Wire Wire Line
 	3200 6150 3350 6150
-NoConn ~ 1400 6150
 NoConn ~ 3200 5750
 NoConn ~ 3200 5850
@@
 	8300 1400 8300 3350
 Wire Wire Line
-	2200 800  2400 800
-Wire Wire Line
-	2400 900  2050 900
-Wire Wire Line
 	4100 2100 4400 2100
 Wire Wire Line
@@
 Wire Wire Line
 	1300 6250 1400 6250
-Wire Wire Line
-	1300 6350 1400 6350
 $Comp
 L Device:Jumper JP1
 U 1 1 5E859075
-P 1300 6650
-F 0 "JP1" V 1346 6562 50  0000 R CNN
-F 1 "Cal" V 1255 6562 50  0000 R CNN
-F 2 "CPB:Socket_Strip_Straight_1x02_Oval_Pitch2.54mm" H 1300 6650 50  0001 C CNN
-F 3 "~" H 1300 6650 50  0001 C CNN
-	1    1300 6650
+P 1050 6600
+F 0 "JP1" V 1096 6512 50  0000 R CNN
+F 1 "Cal" V 1005 6512 50  0000 R CNN
+F 2 "CPB:Socket_Strip_Straight_1x02_Oval_Pitch2.54mm" H 1050 6600 50  0001 C CNN
+F 3 "~" H 1050 6600 50  0001 C CNN
+	1    1050 6600
 	0    -1   -1   0
 $EndComp
-Wire Wire Line
-	1300 6950 1300 7000
-Connection ~ 1300 7000
-Wire Wire Line
-	1300 7000 2300 7000
+$Comp
+L Device:Battery_Cell BT1
+U 1 1 5E862E9B
+P 1050 1050
+F 0 "BT1" V 795 1100 50  0000 C CNN
+F 1 "AA" V 886 1100 50  0000 C CNN
+F 2 "CPB:Battery_Springs_AA" V 1050 1110 50  0001 C CNN
+F 3 "~" V 1050 1110 50  0001 C CNN
+	1    1050 1050
+	0    1    1    0
+$EndComp
+Wire Wire Line
+	1250 1050 1400 1050
+Wire Wire Line
+	950  1050 900  1050
+Wire Wire Line
+	900  1050 900  1300
+$Comp
+L Switch:SW_SPST SW1
+U 1 1 5E86C4A2
+P 1600 1050
+F 0 "SW1" H 1600 825 50  0000 C CNN
+F 1 "POWER" H 1600 916 50  0000 C CNN
+F 2 "CPB:SPST Switch 9mmx3.5mm C223839" H 1600 1050 50  0001 C CNN
+F 3 "" H 1600 1050 50  0001 C CNN
+	1    1600 1050
+	-1   0    0    1
+$EndComp
+Wire Wire Line
+	1800 1050 1950 1050
+Wire Wire Line
+	900  7000 1050 7000
+NoConn ~ 1400 6350
+Wire Wire Line
+	1400 6150 1050 6150
+Wire Wire Line
+	1050 6150 1050 6300
+Wire Wire Line
+	1050 6900 1050 7000
+Connection ~ 1050 7000
+Wire Wire Line
+	1050 7000 2300 7000
 $EndSCHEMATC

Commit message: drop the DS18, switch the MPU to just the four I2C pins, clean up a whole bunch of traces
Parts:
- removed J2: MPU-6050, Connector_PinHeader_2.54mm:PinHeader_1x08_P2.54mm_Vertical, symbol Connector_Generic:Conn_01x08
- removed R4: 1K, Resistor_SMD:R_0805_2012Metric_Pad1.15x1.40mm_HandSolder, symbol Device:R_Small
- removed R8: 10K, Resistor_SMD:R_0805_2012Metric_Pad1.15x1.40mm_HandSolder, symbol Device:R
- removed U3: DS18B20, Package_TO_SOT_THT:TO-92_Inline_Wide, symbol Sensor_Temperature:DS18B20
- added J1: I2C, CPB:Socket_Strip_Straight_1x04_Oval_Pitch2.54mm, symbol Connector_Generic:Conn_01x04
- added R4: 10K, Resistor_SMD:R_0805_2012Metric_Pad1.15x1.40mm_HandSolder, symbol Device:R
- R3: value 4K7 -> 1K; footprint Resistor_SMD:R_0805_2012Metric_Pad1.15x1.40mm_HandSolder -> Resistor_SMD:R_1206_3216Metric_Pad1.42x1.75mm_HandSolder
Connections:
- net labels removed: DQ, EN, GPIO0, GPIO15, GPIO16, RST, VBAT
- wire segments 93 -> 83
- no-connect marks 7 -> 5
Other:
- note added: "NOTE: the MPU-6050\nmodule usually has\nI2C pullups builtin, so we're\nleaving them out here."
- note removed: "Assume the MPU-6050\nmodule has appropriate\nI2C pullups builtin, which\nseems to be typical."
- moved on the sheet: BT1, C1, C6, C7, JP1, R1, R2, R5, R6, SW1, U1

Commit message: looks like we're going to need to switch to an AAA cell if we want this thing to float in such a small container.
Parts:
- BT1: value AA -> NiMH; footprint CPB:Battery_Springs_AA -> CPB:Battery_Springs_AAA
- C7: value 100nF -> 2.2uF
- J1: value I2C -> MPU-6050; footprint CPB:Socket_Strip_Straight_1x04_Oval_Pitch2.54mm -> CPB:MPU-6050 Breakout I2C
Other:
- note added: "10K/2.2uF RC should give\na startup delay of maybe\n25ms. The boost needs extra\ntime to stabilize."
- note added: "Duplicate 10uF caps\nto reduce ESD, as per\ndatasheet. Larger bulk\ncapacitor for 1x NiMH."
- note added: "RST: newer ESP-12F has\ninternal 12k pullup. 47K\nshould allow versions\nwith and without to boot."
- note removed: "Duplicate 10uF caps\nto reduce ESD, as per\ndatasheet. Larger bulk\ncapacitor for 1xAA."
- note removed: "RST: newer ESP-12F has\ninternal 12k pullup"
Changed lines of the file:
@@
 	1    0    0    -1
 $EndComp
-Text Notes 850  5350 0    50   ~ 0
-RST: newer ESP-12F has\ninternal 12k pullup
+Text Notes 850  5450 0    50   ~ 0
+RST: newer ESP-12F has\ninternal 12k pullup. 47K\nshould allow versions\nwith and without to boot.
 $Comp
 L Device:R R5
@@
 P 2200 6800
 F 0 "C7" H 2292 6846 50  0000 L CNN
-F 1 "100nF" H 2292 6755 50  0000 L CNN
+F 1 "2.2uF" H 2292 6755 50  0000 L CNN
 F 2 "Capacitor_SMD:C_0805_2012Metric_Pad1.15x1.40mm_HandSolder" H 2200 6800 50  0001 C CNN
 F 3 "~" H 2200 6800 50  0001 C CNN
@@
 	1650 3050 1650 3000
 Text Notes 3350 3450 0    50   ~ 0
-Duplicate 10uF caps\nto reduce ESD, as per\ndatasheet. Larger bulk\ncapacitor for 1xAA.
+Duplicate 10uF caps\nto reduce ESD, as per\ndatasheet. Larger bulk\ncapacitor for 1x NiMH.
 Wire Wire Line
 	2600 2550 2600 3050
@@
 Wire Wire Line
 	2050 2250 2100 2250
+$Comp
+L Device:Battery_Cell BT1
+U 1 1 5E862E9B
+P 850 900
+F 0 "BT1" V 595 950 50  0000 C CNN
+F 1 "NiMH" V 686 950 50  0000 C CNN
+F 2 "CPB:Battery_Springs_AAA" V 850 960 50  0001 C CNN
+F 3 "~" V 850 960 50  0001 C CNN
+	1    850  900
+	0    1    1    0
+$EndComp
+Wire Wire Line
+	1050 900  1200 900
+Wire Wire Line
+	750  900  700  900
+Wire Wire Line
+	700  900  700  1150
+$Comp
+L Switch:SW_SPST SW1
+U 1 1 5E86C4A2
+P 1400 900
+F 0 "SW1" H 1400 675 50  0000 C CNN
+F 1 "POWER" H 1400 766 50  0000 C CNN
+F 2 "CPB:SPST Switch 9mmx3.5mm C223839" H 1400 900 50  0001 C CNN
+F 3 "" H 1400 900 50  0001 C CNN
+	1    1400 900
+	-1   0    0    1
+$EndComp
+NoConn ~ 2800 6250
+Wire Wire Line
+	2800 6050 2450 6050
+Wire Wire Line
+	2450 6900 3700 6900
+NoConn ~ 2800 6150
+$Comp
+L Connector_Generic:Conn_01x04 J1
+U 1 1 5E97FF96
+P 8300 4750
+F 0 "J1" H 8380 4742 50  0000 L CNN
+F 1 "MPU-6050" H 8380 4651 50  0000 L CNN
+F 2 "CPB:MPU-6050 Breakout I2C" H 8300 4750 50  0001 C CNN
+F 3 "~" H 8300 4750 50  0001 C CNN
+	1    8300 4750
+	1    0    0    -1
+$EndComp
+Wire Wire Line
+	8100 4750 8050 4750
+Wire Wire Line
+	8050 4750 8050 5050
+Wire Wire Line
+	8050 4450 8050 4650
+Wire Wire Line
+	8050 4650 8100 4650
+$Comp
+L power:GND #PWR05
+U 1 1 5E99E221
+P 4350 5050
+F 0 "#PWR05" H 4350 4800 50  0001 C CNN
+F 1 "GND" H 4355 4877 50  0000 C CNN
+F 2 "" H 4350 5050 50  0001 C CNN
+F 3 "" H 4350 5050 50  0001 C CNN
+	1    4350 5050
+	1    0    0    -1
+$EndComp
+Wire Wire Line
+	3700 4950 3950 4950
+Wire Wire Line
+	4150 4950 4350 4950
+Wire Wire Line
+	4350 4950 4350 5050
+$Comp
+L Device:R R7
+U 1 1 5E9A2F33
+P 4700 6650
+F 0 "R7" V 4800 6650 50  0000 C CNN
+F 1 "10K" V 4850 6650 50  0000 C CNN
+F 2 "Resistor_SMD:R_0805_2012Metric_Pad1.15x1.40mm_HandSolder" V 4630 6650 50  0001 C CNN
+F 3 "~" H 4700 6650 50  0001 C CNN
+	1    4700 6650
+	-1   0    0    1
+$EndComp
+Wire Wire Line
+	4700 6250 4700 6500
+Wire Wire Line
+	4700 6800 4700 6900
+Wire Wire Line
+	4700 6900 3700 6900
+$Comp
+L Device:R R4
+U 1 1 5E9A8366
+P 4700 5250
+F 0 "R4" V 4493 5250 50  0000 C CNN
+F 1 "10K" V 4584 5250 50  0000 C CNN
+F 2 "Resistor_SMD:R_0805_2012Metric_Pad1.15x1.40mm_HandSolder" V 4630 5250 50  0001 C CNN
+F 3 "~" H 4700 5250 50  0001 C CNN
+	1    4700 5250
+	-1   0    0    1
+$EndComp
+Wire Wire Line
+	3700 4850 4700 4850
+Wire Wire Line
+	4700 4850 4700 5100
+Wire Wire Line
+	3700 6900 3700 7100
+Connection ~ 3700 4850
+Wire Wire Line
+	3700 4850 3700 4950
+Wire Wire Line
+	4700 5400 4700 6050
+$Comp
+L Device:R_Small R3
+U 1 1 5E9ADDC8
+P 2100 5800
+F 0 "R3" V 2300 5800 50  0000 C CNN
+F 1 "1K" V 2200 5800 50  0000 C CNN
+F 2 "Resistor_SMD:R_1206_3216Metric_Pad1.42x1.75mm_HandSolder" H 2100 5800 50  0001 C CNN
+F 3 "~" H 2100 5800 50  0001 C CNN
+	1    2100 5800
+	-1   0    0    1
+$EndComp
+Wire Wire Line
+	2100 4950 2100 5150
+Wire Wire Line
+	2100 4950 2350 4950
+Wire Wire Line
+	2100 5650 2100 5700
+Wire Wire Line
+	2100 5650 2800 5650
+Wire Wire Line
+	2100 5650 2100 5450
+Connection ~ 2100 5650
+Wire Wire Line
+	2100 5900 2100 5950
+Wire Wire Line
+	2100 5950 2800 5950
+Wire Wire Line
+	2350 5850 2350 5450
+Wire Wire Line
+	2350 5850 2800 5850
+Wire Wire Line
+	2350 5850 2200 5850
+Wire Wire Line
+	2200 5850 2200 6700
+Connection ~ 2350 5850
+Wire Wire Line
+	2200 6900 2450 6900
+Connection ~ 2450 6900
+Wire Wire Line
+	2350 5150 2350 4950
+Connection ~ 2350 4950
+Wire Wire Line
+	2350 4950 3700 4950
+Wire Wire Line
+	3300 2100 3300 1750
+Wire Wire Line
+	3300 1750 2050 1750
+Wire Wire Line
+	2050 1750 2050 2250
+Wire Wire Line
+	1600 900  1650 900
+Wire Wire Line
+	1650 2100 1650 900
+Connection ~ 1650 2100
+Connection ~ 1650 900
+Wire Wire Line
+	1650 900  2550 900
+Wire Wire Line
+	3350 1450 3350 1500
+Connection ~ 3350 1450
+Wire Wire Line
+	7100 4950 8100 4950
+Wire Wire Line
+	7100 4450 8050 4450
+Wire Wire Line
+	7100 4850 8100 4850
+Wire Wire Line
+	2450 6800 2450 6900
+Wire Wire Line
+	2450 6050 2450 6200
 $Comp
 L Device:Jumper JP1
@@
 	0    -1   -1   0
 $EndComp
-$Comp
-L Device:Battery_Cell BT1
-U 1 1 5E862E9B
-P 850 900
-F 0 "BT1" V 595 950 50  0000 C CNN
-F 1 "AA" V 686 950 50  0000 C CNN
-F 2 "CPB:Battery_Springs_AA" V 850 960 50  0001 C CNN
-F 3 "~" V 850 960 50  0001 C CNN
-	1    850  900
-	0    1    1    0
-$EndComp
-Wire Wire Line
-	1050 900  1200 900
-Wire Wire Line
-	750  900  700  900
-Wire Wire Line
-	700  900  700  1150
-$Comp
-L Switch:SW_SPST SW1
-U 1 1 5E86C4A2
-P 1400 900
-F 0 "SW1" H 1400 675 50  0000 C CNN
-F 1 "POWER" H 1400 766 50  0000 C CNN
-F 2 "CPB:SPST Switch 9mmx3.5mm C223839" H 1400 900 50  0001 C CNN
-F 3 "" H 1400 900 50  0001 C CNN
-	1    1400 900
-	-1   0    0    1
-$EndComp
-NoConn ~ 2800 6250
-Wire Wire Line
-	2800 6050 2450 6050
-Wire Wire Line
-	2450 6050 2450 6200
-Wire Wire Line
-	2450 6800 2450 6900
-Wire Wire Line
-	2450 6900 3700 6900
-NoConn ~ 2800 6150
-$Comp
-L Connector_Generic:Conn_01x04 J1
-U 1 1 5E97FF96
-P 8300 4750
-F 0 "J1" H 8380 4742 50  0000 L CNN
-F 1 "I2C" H 8380 4651 50  0000 L CNN
-F 2 "CPB:Socket_Strip_Straight_1x04_Oval_Pitch2.54mm" H 8300 4750 50  0001 C CNN
-F 3 "~" H 8300 4750 50  0001 C CNN
-	1    8300 4750
-	1    0    0    -1
-$EndComp
-Wire Wire Line
-	8100 4750 8050 4750
-Wire Wire Line
-	8050 4750 8050 5050
-Wire Wire Line
-	8050 4450 8050 4650
-Wire Wire Line
-	8050 4650 8100 4650
-$Comp
-L power:GND #PWR05
-U 1 1 5E99E221
-P 4350 5050
-F 0 "#PWR05" H 4350 4800 50  0001 C CNN
-F 1 "GND" H 4355 4877 50  0000 C CNN
-F 2 "" H 4350 5050 50  0001 C CNN
-F 3 "" H 4350 5050 50  0001 C CNN
-	1    4350 5050
-	1    0    0    -1
-$EndComp
-Wire Wire Line
-	3700 4950 3950 4950
-Wire Wire Line
-	4150 4950 4350 4950
-Wire Wire Line
-	4350 4950 4350 5050
-$Comp
-L Device:R R7
-U 1 1 5E9A2F33
-P 4700 6650
-F 0 "R7" V 4800 6650 50  0000 C CNN
-F 1 "10K" V 4850 6650 50  0000 C CNN
-F 2 "Resistor_SMD:R_0805_2012Metric_Pad1.15x1.40mm_HandSolder" V 4630 6650 50  0001 C CNN
-F 3 "~" H 4700 6650 50  0001 C CNN
-	1    4700 6650
-	-1   0    0    1
-$EndComp
-Wire Wire Line
-	4700 6250 4700 6500
-Wire Wire Line
-	4700 6800 4700 6900
-Wire Wire Line
-	4700 6900 3700 6900
-$Comp
-L Device:R R4
-U 1 1 5E9A8366
-P 4700 5250
-F 0 "R4" V 4493 5250 50  0000 C CNN
-F 1 "10K" V 4584 5250 50  0000 C CNN
-F 2 "Resistor_SMD:R_0805_2012Metric_Pad1.15x1.40mm_HandSolder" V 4630 5250 50  0001 C CNN
-F 3 "~" H 4700 5250 50  0001 C CNN
-	1    4700 5250
-	-1   0    0    1
-$EndComp
-Wire Wire Line
-	3700 4850 4700 4850
-Wire Wire Line
-	4700 4850 4700 5100
-Wire Wire Line
-	3700 6900 3700 7100
-Connection ~ 3700 4850
-Wire Wire Line
-	3700 4850 3700 4950
-Wire Wire Line
-	4700 5400 4700 6050
-$Comp
-L Device:R_Small R3
-U 1 1 5E9ADDC8
-P 2100 5800
-F 0 "R3" V 2300 5800 50  0000 C CNN
-F 1 "1K" V 2200 5800 50  0000 C CNN
-F 2 "Resistor_SMD:R_1206_3216Metric_Pad1.42x1.75mm_HandSolder" H 2100 5800 50  0001 C CNN
-F 3 "~" H 2100 5800 50  0001 C CNN
-	1    2100 5800
-	-1   0    0    1
-$EndComp
-Wire Wire Line
-	2100 4950 2100 5150
-Wire Wire Line
-	2100 4950 2350 4950
-Wire Wire Line
-	2100 5650 2100 5700
-Wire Wire Line
-	2100 5650 2800 5650
-Wire Wire Line
-	2100 5650 2100 5450
-Connection ~ 2100 5650
-Wire Wire Line
-	2100 5900 2100 5950
-Wire Wire Line
-	2100 5950 2800 5950
-Wire Wire Line
-	2350 5850 2350 5450
-Wire Wire Line
-	2350 5850 2800 5850
-Wire Wire Line
-	2350 5850 2200 5850
-Wire Wire Line
-	2200 5850 2200 6700
-Connection ~ 2350 5850
-Wire Wire Line
-	2200 6900 2450 6900
-Connection ~ 2450 6900
-Wire Wire Line
-	2350 5150 2350 4950
-Connection ~ 2350 4950
-Wire Wire Line
-	2350 4950 3700 4950
-Wire Wire Line
-	3300 2100 3300 1750
-Wire Wire Line
-	3300 1750 2050 1750
-Wire Wire Line
-	2050 1750 2050 2250
-Wire Wire Line
-	1600 900  1650 900
-Wire Wire Line
-	1650 2100 1650 900
-Connection ~ 1650 2100
-Connection ~ 1650 900
-Wire Wire Line
-	1650 900  2550 900
-Wire Wire Line
-	3350 1450 3350 1500
-Connection ~ 3350 1450
-Wire Wire Line
-	7100 4950 8100 4950
-Wire Wire Line
-	7100 4450 8050 4450
-Wire Wire Line
-	7100 4850 8100 4850
+Text Notes 800  7000 0    50   ~ 0
+10K/2.2uF RC should give\na startup delay of maybe\n25ms. The boost needs extra\ntime to stabilize.
 $EndSCHEMATC

Commit message: a few tweaks
Parts:
- added JP2: REGULATOR, CPB:Jumper 1-2-3 0.5mm, symbol Jumper:Jumper_3_Bridged12
- added U3: MCP1700-3302E_SOT23, Package_TO_SOT_SMD:SOT-23, symbol Regulator_Linear:MCP1700-3302E_SOT23
- C7: value 2.2uF -> 100nF
Connections:
- wire segments 83 -> 91
Other:
- note added: "FIXME: add Li-ion protection"
- note removed: "10K/2.2uF RC should give\na startup delay of maybe\n25ms. The boost needs extra\ntime to stabilize."
- moved on the sheet: C2, C3, C4, C6, R1, R2

Commit message: minor tweaks
Parts:
- JP2: footprint CPB:Jumper 1-2-3 0.5mm -> Jumper:SolderJumper-3_P1.3mm_Bridged12_RoundedPad1.0x1.5mm
Changed lines of the file:
@@
 F 0 "JP2" H 2150 1362 50  0000 C CNN
 F 1 "REGULATOR" H 2150 1453 50  0000 C CNN
-F 2 "CPB:Jumper 1-2-3 0.5mm" H 2150 1250 50  0001 C CNN
+F 2 "Jumper:SolderJumper-3_P1.3mm_Bridged12_RoundedPad1.0x1.5mm" H 2150 1250 50  0001 C CNN
 F 3 "~" H 2150 1250 50  0001 C CNN
 	1    2150 1250

Commit message: a bit of simplifying. We almost certainly don't need that jumper.
Parts:
- removed JP2: REGULATOR, Jumper:SolderJumper-3_P1.3mm_Bridged12_RoundedPad1.0x1.5mm, symbol Jumper:Jumper_3_Bridged12
Connections:
- wire segments 91 -> 90
Other:
- moved on the sheet: C2
Changed lines of the file:
@@
 L Device:C C2
 U 1 1 5CD61C94
-P 2500 2850
-F 0 "C2" H 2588 2896 50  0000 L CNN
-F 1 "10uF" H 2588 2805 50  0000 L CNN
-F 2 "Capacitor_SMD:C_0805_2012Metric_Pad1.15x1.40mm_HandSolder" H 2500 2850 50  0001 C CNN
-F 3 "~" H 2500 2850 50  0001 C CNN
-	1    2500 2850
+P 2400 2550
+F 0 "C2" H 2488 2596 50  0000 L CNN
+F 1 "10uF" H 2488 2505 50  0000 L CNN
+F 2 "Capacitor_SMD:C_0805_2012Metric_Pad1.15x1.40mm_HandSolder" H 2400 2550 50  0001 C CNN
+F 3 "~" H 2400 2550 50  0001 C CNN
+	1    2400 2550
 	1    0    0    -1
 $EndComp
@@
 	1    0    0    -1
 $EndComp
-Wire Wire Line
-	2500 3050 2500 3000
 Text Notes 4200 3450 0    50   ~ 0
 Duplicate 10uF caps\nto reduce ESD, as per\ndatasheet. Larger bulk\ncapacitor for 1x NiMH.
@@
 Wire Wire Line
 	2850 2100 2950 2100
-Wire Wire Line
-	2500 3050 3450 3050
 Wire Wire Line
 	4550 2400 4550 2100
@@
 	1    0    0    -1
 $EndComp
-$Comp
-L Jumper:Jumper_3_Bridged12 JP2
-U 1 1 5E95C87B
-P 2150 1250
-F 0 "JP2" H 2150 1362 50  0000 C CNN
-F 1 "REGULATOR" H 2150 1453 50  0000 C CNN
-F 2 "Jumper:SolderJumper-3_P1.3mm_Bridged12_RoundedPad1.0x1.5mm" H 2150 1250 50  0001 C CNN
-F 3 "~" H 2150 1250 50  0001 C CNN
-	1    2150 1250
-	-1   0    0    1
-$EndComp
-Wire Wire Line
-	1600 900  2150 900
 Wire Wire Line
 	2400 1250 2400 2100
 Wire Wire Line
 	2400 2100 2550 2100
-Wire Wire Line
-	2150 1100 2150 900
-Connection ~ 2150 900
-Wire Wire Line
-	2150 900  2500 900
 Wire Wire Line
 	2050 1750 2900 1750
 Connection ~ 2900 1750
 Wire Wire Line
-	1900 1250 1200 1250
-Wire Wire Line
 	1200 1250 1200 1750
 Wire Wire Line
@@
 Wire Wire Line
 	1750 2050 1750 3050
-Wire Wire Line
-	1750 3050 2500 3050
-Connection ~ 2500 3050
-Wire Wire Line
-	2500 2700 2500 900
-Connection ~ 2500 900
-Wire Wire Line
-	2500 900  3400 900
 Text Notes 900  2100 0    50   ~ 0
 FIXME: add Li-ion protection
 NoConn ~ 4600 5650
 NoConn ~ 4600 5750
+Wire Wire Line
+	1750 3050 2400 3050
+Wire Wire Line
+	2400 2400 2400 2100
+Connection ~ 2400 2100
+Wire Wire Line
+	2400 2700 2400 3050
+Connection ~ 2400 3050
+Wire Wire Line
+	2400 3050 3450 3050
+Wire Wire Line
+	1200 1250 2400 1250
+Wire Wire Line
+	1600 900  2400 900
+Wire Wire Line
+	2400 900  2400 1250
+Connection ~ 2400 900
+Wire Wire Line
+	2400 900  3400 900
+Connection ~ 2400 1250
 $EndSCHEMATC

Commit message: simpler, shorter version that uses lipo battery pack with JST-PH2.0 connectors
Parts:
- removed C4: 10uF, Capacitor_SMD:C_0805_2012Metric_Pad1.15x1.40mm_HandSolder, symbol Device:C
- removed C5: 100uF, Capacitor_Tantalum_SMD:CP_EIA-3528-12_Kemet-T_Pad1.50x2.35mm_HandSolder, symbol Device:CP1_Small
- removed L1: 10uH, Inductor_SMD:L_Coilcraft_XxL4040, symbol Device:L
- removed U2: HT7733SA, Package_TO_SOT_SMD:SOT-23-5, symbol Holtek:HT7733SA
- added C4: 100nF, Capacitor_SMD:C_0805_2012Metric_Pad1.15x1.40mm_HandSolder, symbol Device:C_Small
- added R8: 100R, Resistor_SMD:R_0805_2012Metric_Pad1.15x1.40mm_HandSolder, symbol Device:R_Small
- added U2: BRCL3130MC, Package_TO_SOT_SMD:SOT-23_Handsoldering, symbol Blue~Rocket:BRCL3130MC
- BT1: value NiMH -> Li 3.7v; footprint CPB:Battery_Springs_AAA -> Connector_JST:JST_PH_S2B-PH-K_1x02_P2.00mm_Horizontal
- C3: value 10uF -> 22uF
- U3: value MCP1700-3302E_SOT23 -> HT7333; footprint Package_TO_SOT_SMD:SOT-23 -> Package_TO_SOT_SMD:SOT-23_Handsoldering
Connections:
- wire segments 90 -> 83
Other:
- note removed: "Duplicate 10uF caps\nto reduce ESD, as per\ndatasheet. Larger bulk\ncapacitor for 1x NiMH."
- note removed: "FIXME: add Li-ion protection"
- moved on the sheet: BT1, C2, C3, C6, R1, R2, SW1, U3
