File: weeSpindel.sch (KiCad schematic (older format))
At the start: 21 parts, among them J1 MPU-6050, SW1 POWER, U1 ESP-12E, U2 BRCL3130MC, U3 HT7333

Commit message: progress on a smaller version using a JST-PH lipo cell off the end
Parts:
- U3: value HT7333 -> HT7233
Changed lines of the file:
@@
 	1    0    0    -1
 $EndComp
-Text Notes 850  5450 0    50   ~ 0
+Text Notes 750  5450 0    50   ~ 0
 RST: newer ESP-12F has\ninternal 12k pullup. 47K\nshould allow versions\nwith and without to boot.
 $Comp
@@
 P 2100 5300
 F 0 "R5" V 2200 5300 50  0000 C CNN
-F 1 "47K" V 2250 5300 50  0000 C CNN
+F 1 "47K" V 2300 5300 50  0000 C CNN
 F 2 "Resistor_SMD:R_0805_2012Metric_Pad1.15x1.40mm_HandSolder" V 2030 5300 50  0001 C CNN
 F 3 "~" H 2100 5300 50  0001 C CNN
@@
 P 4700 6650
 F 0 "R7" V 4800 6650 50  0000 C CNN
-F 1 "10K" V 4850 6650 50  0000 C CNN
+F 1 "10K" V 4900 6650 50  0000 C CNN
 F 2 "Resistor_SMD:R_0805_2012Metric_Pad1.15x1.40mm_HandSolder" V 4630 6650 50  0001 C CNN
 F 3 "~" H 4700 6650 50  0001 C CNN
@@
 P 4200 2500
 F 0 "U3" H 4200 2742 50  0000 C CNN
-F 1 "HT7333" H 4200 2651 50  0000 C CNN
+F 1 "HT7233" H 4200 2651 50  0000 C CNN
 F 2 "Package_TO_SOT_SMD:SOT-23_Handsoldering" H 4200 2725 50  0001 C CNN
 F 3 "http://ww1.microchip.com/downloads/en/DeviceDoc/20001826C.pdf" H 4200 2500 50  0001 C CNN

Commit message: add USB programming
Parts:
- removed C7: 100nF, Capacitor_SMD:C_0805_2012Metric_Pad1.15x1.40mm_HandSolder, symbol Device:C_Small
- added C5, C8: 100nF, Capacitor_SMD:C_0603_1608Metric_Pad1.05x0.95mm_HandSolder, symbol Device:C_Small
- added D1: B5817WL, Diode_SMD:D_SOD-123F, symbol Device:D_Schottky
- added F1: 350mA, Fuse:Fuse_0805_2012Metric_Pad1.15x1.40mm_HandSolder, symbol Device:Polyfuse_Small
- added J2: USB_B_Micro, CPB:USB Micro-B C10418, symbol Connector:USB_B_Micro
- added R9: 470R, Resistor_SMD:R_0805_2012Metric_Pad1.15x1.40mm_HandSolder, symbol Device:R_Small
- added SW2: RESET, Button_Switch_SMD:SW_SPST_CK_RS282G05A3, symbol Switch:SW_Push
- added SW3: PROG, Button_Switch_SMD:SW_SPST_CK_RS282G05A3, symbol Switch:SW_Push
- added U4: CH330N, Package_SO:SOIC-8_3.9x4.9mm_P1.27mm, symbol Interface_USB:CH330N
- C1, C4, C6: footprint Capacitor_SMD:C_0805_2012Metric_Pad1.15x1.40mm_HandSolder -> Capacitor_SMD:C_0603_1608Metric_Pad1.05x0.95mm_HandSolder
- R3: footprint Resistor_SMD:R_1206_3216Metric_Pad1.42x1.75mm_HandSolder -> Resistor_SMD:R_0805_2012Metric_Pad1.15x1.40mm_HandSolder
- R4, R5, R6, R7: footprint Resistor_SMD:R_0805_2012Metric_Pad1.15x1.40mm_HandSolder -> Resistor_SMD:R_0603_1608Metric_Pad1.05x0.95mm_HandSolder
Connections:
- net labels added: +5V, eRX, eTX
- wire segments 83 -> 117

Commit message: add support for both li-ion and NiMH/Alkaline chemistries, plus USB programming. Among other things.
Parts:
- D1: footprint Diode_SMD:D_SOD-123F -> Diode_SMD:D_SOD-323F
- F1: footprint Fuse:Fuse_0805_2012Metric_Pad1.15x1.40mm_HandSolder -> Fuse:Fuse_0603_1608Metric_Pad1.05x0.95mm_HandSolder
- R1, R2, R3, R8, R9: footprint Resistor_SMD:R_0805_2012Metric_Pad1.15x1.40mm_HandSolder -> Resistor_SMD:R_0603_1608Metric_Pad1.05x0.95mm_HandSolder
Changed lines of the file:
@@
 F 0 "R1" V 4093 1300 50  0000 C CNN
 F 1 "1M" V 4184 1300 50  0000 C CNN
-F 2 "Resistor_SMD:R_0805_2012Metric_Pad1.15x1.40mm_HandSolder" V 4230 1300 50  0001 C CNN
+F 2 "Resistor_SMD:R_0603_1608Metric_Pad1.05x0.95mm_HandSolder" V 4230 1300 50  0001 C CNN
 F 3 "~" H 4300 1300 50  0001 C CNN
 	1    4300 1300
@@
 F 0 "R2" H 4530 1604 50  0000 R CNN
 F 1 "330K" H 4530 1695 50  0000 R CNN
-F 2 "Resistor_SMD:R_0805_2012Metric_Pad1.15x1.40mm_HandSolder" V 4530 1650 50  0001 C CNN
+F 2 "Resistor_SMD:R_0603_1608Metric_Pad1.05x0.95mm_HandSolder" V 4530 1650 50  0001 C CNN
 F 3 "~" H 4600 1650 50  0001 C CNN
 	1    4600 1650
@@
 F 0 "R3" V 2300 5800 50  0000 C CNN
 F 1 "1K" V 2200 5800 50  0000 C CNN
-F 2 "Resistor_SMD:R_0805_2012Metric_Pad1.15x1.40mm_HandSolder" H 2100 5800 50  0001 C CNN
+F 2 "Resistor_SMD:R_0603_1608Metric_Pad1.05x0.95mm_HandSolder" H 2100 5800 50  0001 C CNN
 F 3 "~" H 2100 5800 50  0001 C CNN
 	1    2100 5800
@@
 F 0 "R8" H 2409 2296 50  0000 L CNN
 F 1 "100R" H 2409 2205 50  0000 L CNN
-F 2 "Resistor_SMD:R_0805_2012Metric_Pad1.15x1.40mm_HandSolder" H 2350 2250 50  0001 C CNN
+F 2 "Resistor_SMD:R_0603_1608Metric_Pad1.05x0.95mm_HandSolder" H 2350 2250 50  0001 C CNN
 F 3 "~" H 2350 2250 50  0001 C CNN
 	1    2350 2250
@@
 F 0 "F1" H 2418 1696 50  0000 L CNN
 F 1 "350mA" H 2418 1605 50  0000 L CNN
-F 2 "Fuse:Fuse_0805_2012Metric_Pad1.15x1.40mm_HandSolder" H 2400 1450 50  0001 L CNN
+F 2 "Fuse:Fuse_0603_1608Metric_Pad1.05x0.95mm_HandSolder" H 2400 1450 50  0001 L CNN
 F 3 "~" H 2350 1650 50  0001 C CNN
 	1    2350 1650
@@
 F 0 "D1" H 8300 834 50  0000 C CNN
 F 1 "B5817WL" H 8300 925 50  0000 C CNN
-F 2 "Diode_SMD:D_SOD-123F" H 8300 1050 50  0001 C CNN
+F 2 "Diode_SMD:D_SOD-323F" H 8300 1050 50  0001 C CNN
 F 3 "~" H 8300 1050 50  0001 C CNN
 	1    8300 1050
@@
 F 0 "R9" V 8854 1700 50  0000 C CNN
 F 1 "470R" V 8945 1700 50  0000 C CNN
-F 2 "Resistor_SMD:R_0805_2012Metric_Pad1.15x1.40mm_HandSolder" H 9050 1700 50  0001 C CNN
+F 2 "Resistor_SMD:R_0603_1608Metric_Pad1.05x0.95mm_HandSolder" H 9050 1700 50  0001 C CNN
 F 3 "~" H 9050 1700 50  0001 C CNN
 	1    9050 1700
