File: weeSpindel.kicad_sch (KiCad schematic)
At the start: 37 parts, among them J1 MPU-6050, J2 USB_B_Micro, SW2 RESET, SW3 PROG, U1 ESP-12E, U2 BRCL3130MC, U3 HT7233, U4 CH330N, U5 HT7733SA

Commit message: some more tidying. ground plane is actually more of a plane now.
Parts:
- R3: value 1K -> 470R
Connections:
- net EN: now also SW2.1
- net RST: no longer SW2.1
Changed lines of the file:
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@@
   (junction (at 38.1 102.87) (diameter 0) (color 0 0 0 0)
+  )
+  (junction (at 198.755 122.555) (diameter 0) (color 0 0 0 0)
   )
   (junction (at 58.42 141.605) (diameter 0) (color 0 0 0 0)
@@
     (stroke (width 0) (type default) (color 0 0 0 0))
   )
-  (wire (pts (xy 180.975 113.665) (xy 180.975 127.635))
-    (stroke (width 0) (type default) (color 0 0 0 0))
-  )
   (wire (pts (xy 259.715 121.285) (xy 255.905 121.285))
     (stroke (width 0) (type default) (color 0 0 0 0))
@@
     (stroke (width 0) (type default) (color 0 0 0 0))
   )
+  (wire (pts (xy 180.975 122.555) (xy 198.755 122.555))
+    (stroke (width 0) (type default) (color 0 0 0 0))
+  )
   (wire (pts (xy 168.91 57.15) (xy 166.37 57.15))
     (stroke (width 0) (type default) (color 0 0 0 0))
@@
     (stroke (width 0) (type default) (color 0 0 0 0))
   )
-  (wire (pts (xy 198.755 118.745) (xy 198.755 123.19))
+  (wire (pts (xy 198.755 118.745) (xy 198.755 122.555))
     (stroke (width 0) (type default) (color 0 0 0 0))
   )
@@
     (stroke (width 0) (type default) (color 0 0 0 0))
   )
-  (wire (pts (xy 192.405 113.665) (xy 180.975 113.665))
-    (stroke (width 0) (type default) (color 0 0 0 0))
-  )
   (wire (pts (xy 176.53 48.26) (xy 204.47 48.26))
     (stroke (width 0) (type default) (color 0 0 0 0))
@@
     (stroke (width 0) (type default) (color 0 0 0 0))
   )
+  (wire (pts (xy 180.975 122.555) (xy 180.975 127.635))
+    (stroke (width 0) (type default) (color 0 0 0 0))
+  )
   (wire (pts (xy 49.53 127.635) (xy 58.42 127.635))
     (stroke (width 0) (type default) (color 0 0 0 0))
@@
   )
   (wire (pts (xy 168.91 57.15) (xy 168.91 55.88))
+    (stroke (width 0) (type default) (color 0 0 0 0))
+  )
+  (wire (pts (xy 198.755 122.555) (xy 198.755 123.19))
     (stroke (width 0) (type default) (color 0 0 0 0))
   )
@@
     (in_bom yes) (on_board yes)
     (property "Reference" "R3" (id 0) (at 187.325 117.475 90))
-    (property "Value" "1K" (id 1) (at 189.865 117.475 90))
+    (property "Value" "470R" (id 1) (at 189.865 117.475 90))
     (property "Footprint" "Resistor_SMD:R_0603_1608Metric_Pad0.98x0.95mm_HandSolder" (id 2) (at 192.405 117.475 0)
       (effects (font (size 1.27 1.27)) hide)
@@
     )
     (path "/00000000-0000-0000-0000-00005e9addc8"
-      (reference "R3") (unit 1) (value "1K") (footprint "Resistor_SMD:R_0603_1608Metric_Pad0.98x0.95mm_HandSolder")
+      (reference "R3") (unit 1) (value "470R") (footprint "Resistor_SMD:R_0603_1608Metric_Pad0.98x0.95mm_HandSolder")
     )
     (path "/00000000-0000-0000-0000-00005e9a8366"
